File: PowerSupply.kicad_pcb (KiCad board)
At the start: 2 copper layers, 1 part

Commit message: adddd
Parts:
- added REF**: Elko_vert_11.2x6.3mm_RM2.5_CopperClear, Capacitors_Elko_ThroughHole:Elko_vert_11.2x6.3mm_RM2.5_CopperClear, F.Cu at (194.3, 125.7)
- added REF**: DIP-22_W10.16mm_LongPads, Housings_DIP:DIP-22_W10.16mm_LongPads, F.Cu at (92.7, 133.3)
Routing:
- net (no net): track 0.00 -> 142.2 mm
Changed lines of the file:
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@@
     (links 0)
     (no_connects 0)
-    (area 0 0 0 0)
+    (area 117.615713 101.618 165.594287 134.071)
     (thickness 1.6)
     (drawings 0)
-    (tracks 0)
+    (tracks 15)
     (zones 0)
-    (modules 1)
+    (modules 3)
     (nets 1)
   )
@@
     (pad_to_mask_clearance 0)
     (aux_axis_origin 0 0)
-    (visible_elements FFFFF77F)
+    (visible_elements 7FFFFFFF)
     (pcbplotparams
       (layerselection 0x00030_80000001)
@@
     (pad 2 thru_hole circle (at -12.065 0) (size 5.00126 5.00126) (drill 2.79908) (layers *.Cu *.Mask F.SilkS))
   )
+  (module Capacitors_Elko_ThroughHole:Elko_vert_11.2x6.3mm_RM2.5_CopperClear (layer F.Cu)
+    (at 194.31 125.73)
+    (descr "Electrolytic Capacitor, vertical, diameter 6,3mm, RM 2,5mm, CopperClear, radial,")
+    (tags "Electrolytic Capacitor, vertical, diameter 6,3mm, RM 2,5mm, Elko, Electrolytkondensator, Kondensator gepolt, Durchmesser 6,3mm, CopperClear, radial,")
+    (fp_text reference REF** (at 1.27 -5.08) (layer F.SilkS)
+      (effects (font (size 1 1) (thickness 0.15)))
+    )
+    (fp_text value Elko_vert_11.2x6.3mm_RM2.5_CopperClear (at 1.27 5.08) (layer F.Fab)
+      (effects (font (size 1 1) (thickness 0.15)))
+    )
+    (fp_line (start 0.26924 -1.69926) (end 0.76962 -1.69926) (layer F.SilkS) (width 0.15))
+    (fp_line (start 0.26924 -1.69926) (end 0.26924 -2.19964) (layer F.SilkS) (width 0.15))
+    (fp_line (start -0.23114 -1.69926) (end 0.26924 -1.69926) (layer F.SilkS) (width 0.15))
+    (fp_line (start 0.26924 -1.69926) (end 0.26924 -1.30048) (layer F.SilkS) (width 0.15))
+    (fp_line (start 0.26924 -1.30048) (end 0.26924 -1.19888) (layer F.SilkS) (width 0.15))
+    (fp_circle (center 1.27 0) (end 4.4196 0) (layer F.SilkS) (width 0.15))
+    (pad 2 thru_hole circle (at 2.54 0) (size 1.50114 1.50114) (drill 0.8001) (layers *.Cu *.Mask F.SilkS))
+    (pad 1 thru_hole circle (at 0 0) (size 1.50114 1.50114) (drill 0.8001) (layers *.Cu *.Mask F.SilkS))
+    (model Capacitors_Elko_ThroughHole.3dshapes/Elko_vert_11.2x6.3mm_RM2.5_CopperClear.wrl
+      (at (xyz 0 0 0))
+      (scale (xyz 1 1 1))
+      (rotate (xyz 0 0 0))
+    )
+  )
+  (module Housings_DIP:DIP-22_W10.16mm_LongPads (layer F.Cu)
+    (at 92.71 133.35)
+    (descr "22-lead dip package, row spacing 10.16 mm (400 mils), longer pads")
+    (tags "dil dip 2.54 400")
+    (fp_text reference REF** (at 0 -5.22) (layer F.SilkS)
+      (effects (font (size 1 1) (thickness 0.15)))
+    )
+    (fp_text value DIP-22_W10.16mm_LongPads (at 0 -3.72) (layer F.Fab)
+      (effects (font (size 1 1) (thickness 0.15)))
+    )
+    (fp_line (start -1.4 -2.45) (end -1.4 27.85) (layer F.CrtYd) (width 0.05))
+    (fp_line (start 11.55 -2.45) (end 11.55 27.85) (layer F.CrtYd) (width 0.05))
+    (fp_line (start -1.4 -2.45) (end 11.55 -2.45) (layer F.CrtYd) (width 0.05))
+    (fp_line (start -1.4 27.85) (end 11.55 27.85) (layer F.CrtYd) (width 0.05))
+    (fp_line (start 0.135 -2.295) (end 0.135 -1.025) (layer F.SilkS) (width 0.15))
+    (fp_line (start 10.025 -2.295) (end 10.025 -1.025) (layer F.SilkS) (width 0.15))
+    (fp_line (start 10.025 27.695) (end 10.025 26.425) (layer F.SilkS) (width 0.15))
+    (fp_line (start 0.135 27.695) (end 0.135 26.425) (layer F.SilkS) (width 0.15))
+    (fp_line (start 0.135 -2.295) (end 10.025 -2.295) (layer F.SilkS) (width 0.15))
+    (fp_line (start 0.135 27.695) (end 10.025 27.695) (layer F.SilkS) (width 0.15))
+    (fp_line (start 0.135 -1.025) (end -1.15 -1.025) (layer F.SilkS) (width 0.15))
+    (pad 1 thru_hole oval (at 0 0) (size 2.3 1.6) (drill 0.8) (layers *.Cu *.Mask F.SilkS))
+    (pad 2 thru_hole oval (at 0 2.54) (size 2.3 1.6) (drill 0.8) (layers *.Cu *.Mask F.SilkS))
+    (pad 3 thru_hole oval (at 0 5.08) (size 2.3 1.6) (drill 0.8) (layers *.Cu *.Mask F.SilkS))
+    (pad 4 thru_hole oval (at 0 7.62) (size 2.3 1.6) (drill 0.8) (layers *.Cu *.Mask F.SilkS))
+    (pad 5 thru_hole oval (at 0 10.16) (size 2.3 1.6) (drill 0.8) (layers *.Cu *.Mask F.SilkS))
+    (pad 6 thru_hole oval (at 0 12.7) (size 2.3 1.6) (drill 0.8) (layers *.Cu *.Mask F.SilkS))
+    (pad 7 thru_hole oval (at 0 15.24) (size 2.3 1.6) (drill 0.8) (layers *.Cu *.Mask F.SilkS))
+    (pad 8 thru_hole oval (at 0 17.78) (size 2.3 1.6) (drill 0.8) (layers *.Cu *.Mask F.SilkS))
+    (pad 9 thru_hole oval (at 0 20.32) (size 2.3 1.6) (drill 0.8) (layers *.Cu *.Mask F.SilkS))
+    (pad 10 thru_hole oval (at 0 22.86) (size 2.3 1.6) (drill 0.8) (layers *.Cu *.Mask F.SilkS))
+    (pad 11 thru_hole oval (at 0 25.4) (size 2.3 1.6) (drill 0.8) (layers *.Cu *.Mask F.SilkS))
+    (pad 12 thru_hole oval (at 10.16 25.4) (size 2.3 1.6) (drill 0.8) (layers *.Cu *.Mask F.SilkS))
+    (pad 13 thru_hole oval (at 10.16 22.86) (size 2.3 1.6) (drill 0.8) (layers *.Cu *.Mask F.SilkS))
+    (pad 14 thru_hole oval (at 10.16 20.32) (size 2.3 1.6) (drill 0.8) (layers *.Cu *.Mask F.SilkS))
+    (pad 15 thru_hole oval (at 10.16 17.78) (size 2.3 1.6) (drill 0.8) (layers *.Cu *.Mask F.SilkS))
+    (pad 16 thru_hole oval (at 10.16 15.24) (size 2.3 1.6) (drill 0.8) (layers *.Cu *.Mask F.SilkS))
+    (pad 17 thru_hole oval (at 10.16 12.7) (size 2.3 1.6) (drill 0.8) (layers *.Cu *.Mask F.SilkS))
+    (pad 18 thru_hole oval (at 10.16 10.16) (size 2.3 1.6) (drill 0.8) (layers *.Cu *.Mask F.SilkS))
+    (pad 19 thru_hole oval (at 10.16 7.62) (size 2.3 1.6) (drill 0.8) (layers *.Cu *.Mask F.SilkS))
+    (pad 20 thru_hole oval (at 10.16 5.08) (size 2.3 1.6) (drill 0.8) (layers *.Cu *.Mask F.SilkS))
+    (pad 21 thru_hole oval (at 10.16 2.54) (size 2.3 1.6) (drill 0.8) (layers *.Cu *.Mask F.SilkS))
+    (pad 22 thru_hole oval (at 10.16 0) (size 2.3 1.6) (drill 0.8) (layers *.Cu *.Mask F.SilkS))
+    (model Housings_DIP.3dshapes/DIP-22_W10.16mm_LongPads.wrl
+      (at (xyz 0 0 0))
+      (scale (xyz 1 1 1))
+      (rotate (xyz 0 0 0))
+    )
+  )
+  (segment (start 113.03 137.16) (end 124.46 125.73) (width 0.25) (layer B.Cu) (net 0))
+  (segment (start 99.06 133.35) (end 102.87 137.16) (width 0.25) (layer B.Cu) (net 0))
+  (segment (start 102.87 137.16) (end 113.03 137.16) (width 0.25) (layer B.Cu) (net 0))
+  (segment (start 100.33 132.08) (end 99.06 133.35) (width 0.25) (layer B.Cu) (net 0))
+  (segment (start 106.68 128.27) (end 102.87 132.08) (width 0.25) (layer B.Cu) (net 0))
+  (segment (start 102.87 132.08) (end 100.33 132.08) (width 0.25) (layer B.Cu) (net 0))
+  (segment (start 110.13005 124.81995) (end 106.68 128.27) (width 0.25) (layer B.Cu) (net 0))
+  (segment (start 110.13005 133.35) (end 112.395 133.35) (width 0.25) (layer B.Cu) (net 0))
+  (segment (start 102.87 133.35) (end 110.13005 133.35) (width 0.25) (layer B.Cu) (net 0))
+  (segment (start 110.13005 133.35) (end 110.13005 124.81995) (width 0.25) (layer B.Cu) (net 0))
+  (segment (start 104.49 134.62) (end 135.255 134.62) (width 0.25) (layer B.Cu) (net 0))
+  (segment (start 135.255 134.62) (end 151.765 118.11) (width 0.25) (layer B.Cu) (net 0))
+  (segment (start 102.87 135.89) (end 103.22 135.89) (width 0.25) (layer B.Cu) (net 0))
+  (segment (start 103.22 135.89) (end 104.49 134.62) (width 0.25) (layer B.Cu) (net 0))
+  (segment (start 112.395 133.35) (end 127.635 118.11) (width 0.25) (layer B.Cu) (net 0))
 )
